File: VIC-20-InternalRAM.kicad_pcb (KiCad board)
At the start: 2 copper layers, 103 x 40.8 mm, 11 parts, among them J1 P6, SW1 SW_DIP_x04, U1 CY6264-70SNC, U2 CY6264-70SNC, U3 CY6264-70SNC, U4 CY6264-70SNC, U5 27C64 - BASIC, U6 27C64 - KERNEL, U7 BASIC, U8 KERNEL

Commit message: update render
Other:
- board text added: "VIC 20 ROM Replacement + Internal RAM Expansion Design by Julian Brown 2024 CC BY-NC-SA 4.0"
- board text removed: "VIC 20 ROM Replacement + Internal RAM Expansion Design by Julian Brown 2024"
Changed lines of the file:
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@@
 		)
 	)
-	(gr_text "VIC 20 ROM Replacement\n+\nInternal RAM Expansion\nDesign by Julian Brown 2024"
-		(at 142.5194 101.1428 0)
+	(gr_text "VIC 20 ROM Replacement\n+\nInternal RAM Expansion\nDesign by Julian Brown 2024\nCC BY-NC-SA 4.0"
+		(at 142.7988 95.123 0)
 		(layer "F.SilkS")
 		(effects
@@
 				(thickness 0.1)
 			)
-			(justify left bottom)
+			(justify left top)
 		)
 	)
